Commit message: feat: qualify E0-v2 servo action contract

File: source/base_locomotion_stackforce_quadrupedal/base_locomotion_stackforce_quadrupedal/assets/robots/stackforce_quadrupedal_wheeled_robot/urdf/stackforce_quadrupedal_wheeled_robot.urdf (robot description, URDF)
Before this commit: robot stackforce_quadrupedal_wheeled_robot, 29 links, 28 joints
Joints:
- joint FL_Outer_Knee_Joint: limit lower=-1.57 upper=1.57 effort=0.392 velocity=8.73 -> lower=-3.14159265359 upper=3.14159265359 effort=0.392 velocity=8.73
- joint FR_Outer_Knee_Joint: limit lower=-1.57 upper=1.57 effort=0.392 velocity=8.73 -> lower=-3.14159265359 upper=3.14159265359 effort=0.392 velocity=8.73
- joint RL_Outer_Knee_Joint: limit lower=-1.57 upper=1.57 effort=0.392 velocity=8.73 -> lower=-3.14159265359 upper=3.14159265359 effort=0.392 velocity=8.73
- joint RR_Outer_Knee_Joint: limit lower=-1.57 upper=1.57 effort=0.392 velocity=8.73 -> lower=-3.14159265359 upper=3.14159265359 effort=0.392 velocity=8.73
